Commit message: remove sdf file and modify urdf file

File: armmy_turtlebot3/urdf/turtlebot3_burger_custom.urdf (robot description, URDF)
Before this commit: robot turtlebot3_burger, 8 links, 7 joints
Links:
- link arm_link: mass None -> 0.1; geometry collision box size=0.15 0.01 0.01; visual box size=0.15 0.01 0.01
Joints:
- joint arm_joint: origin xyz=0 0 0.181 rpy=0 0 0 -> xyz=0 0 0.201 rpy=0 0 0; parent base_link -> base_footprint

Commit message: add articubot for ref, need to fix slower rotate in gazebo. (turtlebot3 issue only, articubot is normaly might have issue with tb3 urdf config(inertial or ...))

File: armmy_turtlebot3/urdf/turtlebot3_burger_custom.urdf (robot description, URDF)
Before this commit: robot turtlebot3_burger_custom, 8 links, 7 joints
Links:
- removed link arm_link
- link base_link: mass 8.2573504e-01 -> 0.1
- link wheel_left_link: geometry collision sphere radius=0.033; visual mesh filename=package://turtlebot3_gazebo/models/turtlebot3_common/meshes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 scale=0.001 0.001 0.001
- link wheel_right_link: geometry collision sphere radius=0.033; visual mesh filename=package://turtlebot3_gazebo/models/turtlebot3_common/meshes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 scale=0.001 0.001 0.001
Joints:
- removed joint arm_joint
