Commit message: fix lidar frame_name in xarco file

File: armmy_turtlebot3/urdf/articubot/camera.xacro (robot description, xacro)
@@ -2,5 +2,5 @@
 <robot xmlns:xacro="http://www.ros.org/wiki/xacro" >
     <joint name="camera_joint" type="fixed">
-        <parent link="chassis"/>
+        <parent link="base_link"/>
         <child link="camera_link"/>
         <origin xyz="0.276 0 0.181" rpy="0 0.18 0"/>

File: armmy_turtlebot3/urdf/articubot/depth_camera.xacro (robot description, xacro)
@@ -2,5 +2,5 @@
 <robot xmlns:xacro="http://www.ros.org/wiki/xacro" >
     <joint name="camera_joint" type="fixed">
-        <parent link="chassis"/>
+        <parent link="base_link"/>
         <child link="camera_link"/>
         <origin xyz="0.305 0 0.08" rpy="0 0 0"/>

File: armmy_turtlebot3/urdf/articubot/face.xacro (robot description, xacro)
@@ -2,5 +2,5 @@
 <robot xmlns:xacro="http://www.ros.org/wiki/xacro" >
     <joint name="face_joint" type="fixed">
-        <parent link="chassis"/>
+        <parent link="base_link"/>
         <child link="face_link"/>
         <origin xyz="${chassis_length} 0 ${chassis_height/2}" rpy="0 0 0"/>

File: armmy_turtlebot3/urdf/articubot/lidar.xacro (robot description, xacro)
@@ -2,5 +2,5 @@
 <robot xmlns:xacro="http://www.ros.org/wiki/xacro" >
     <joint name="laser_joint" type="fixed">
-        <parent link="chassis"/>
+        <parent link="base_link"/>
         <child link="laser_frame"/>
         <origin xyz="0.122 0 0.212" rpy="0 0 0"/>

File: armmy_turtlebot3/urdf/tb3_custom/gazebo_control.xacro (robot description, xacro)
@@ -4,6 +4,6 @@
         <plugin name="diff_drive" filename="libgazebo_ros_diff_drive.so">
             <!-- Wheel Information -->
-            <left_joint>left_wheel_joint</left_joint>
-            <right_joint>right_wheel_joint</right_joint>
+            <left_joint>wheel_left_joint</left_joint>
+            <right_joint>wheel_right_joint</right_joint>
             <wheel_separation>0.297</wheel_separation>
             <wheel_diameter>0.066</wheel_diameter>

File: armmy_turtlebot3/urdf/tb3_custom/lidar.xacro (robot description, xacro)
@@ -58,5 +58,5 @@
                 </ros>
                 <output_type>sensor_msgs/LaserScan</output_type>
-                <frame_name>base_scan</frame_name>
+                <frame_name>laser_frame</frame_name>
             </plugin>
         </sensor>

File: armmy_turtlebot3/urdf/tb3_custom/ros2_control.xacro (robot description, xacro)
@@ -55,5 +55,5 @@
                 <command_interface name="position"/>
                 <state_interface name="position">
-                  <param name="initial_value">0.15</param>
+                  <param name="initial_value">0.0</param>
                 </state_interface>
                 <state_interface name="velocity"/>
