Commit message: fix tf from base_link -> base_footprint

File: armmy_turtlebot3/urdf/tb3_custom/gazebo_control.xacro (robot description, xacro)
@@ -14,5 +14,5 @@
             <!-- Output -->
             <odometry_frame>odom</odometry_frame>
-            <robot_base_frame>base_link</robot_base_frame>
+            <robot_base_frame>base_footprint</robot_base_frame>
             <publish_odom>true</publish_odom>
             <publish_odom_tf>true</publish_odom_tf>

File: armmy_turtlebot3/urdf/tb3_custom/lidar.xacro (robot description, xacro)
@@ -10,5 +10,5 @@
             <origin xyz="0 0 0.0" rpy="0 0 0" />
             <geometry>
-                <mesh filename="package://turtlebot3_gazebo/models/turtlebot3_common/meshes/lds.dae"
+                <mesh filename="package://turtlebot3_common/meshes/lds.dae"
                     scale="0.001 0.001 0.001" />
             </geometry>

File: armmy_turtlebot3/urdf/tb3_custom/robot_core.xacro (robot description, xacro)
@@ -58,5 +58,5 @@
             <geometry>
                 <mesh
-                    filename="package://turtlebot3_gazebo/models/turtlebot3_common/meshes/burger_base.dae"
+                    filename="package://turtlebot3_common/meshes/burger_base.dae"
                     scale="0.001 0.001 0.001" />
             </geometry>
@@ -85,5 +85,5 @@
             <geometry>
                 <mesh
-                    filename="package://turtlebot3_gazebo/models/turtlebot3_common/meshes/tire.dae"
+                    filename="package://turtlebot3_common/meshes/tire.dae"
                     scale="0.001 0.001 0.001" />
             </geometry>
@@ -112,5 +112,5 @@
             <geometry>
                 <mesh
-                    filename="package://turtlebot3_gazebo/models/turtlebot3_common/meshes/tire.dae"
+                    filename="package://turtlebot3_common/meshes/tire.dae"
                     scale="0.001 0.001 0.001" />
             </geometry>

File: armmy_turtlebot3/urdf/tb3_custom/ros2_control.xacro (robot description, xacro)
@@ -69,5 +69,5 @@
             </ros>
             <parameters>$(find armmy_turtlebot3)/config/ros2_controller/my_controllers.yaml</parameters>
-            <parameters>$(find armmy_turtlebot3)/config/ros2_controller/gaz_ros2_ctl_use_sim.yaml</parameters>
+            <!-- <parameters>$(find armmy_turtlebot3)/config/ros2_controller/gaz_ros2_ctl_use_sim.yaml</parameters> -->
         </plugin>
     </gazebo>
