Commit message: fix model not loading in RVIZ

File: armmy_turtlebot3/urdf/tb3_custom/lidar.xacro (robot description, xacro)
@@ -10,5 +10,5 @@
             <origin xyz="0 0 0.0" rpy="0 0 0" />
             <geometry>
-                <mesh filename="package://turtlebot3_common/meshes/lds.dae"
+                <mesh filename="package://armmy_turtlebot3/models/turtlebot3_common//meshes/lds.dae"
                     scale="0.001 0.001 0.001" />
             </geometry>

File: armmy_turtlebot3/urdf/tb3_custom/robot_core.xacro (robot description, xacro)
@@ -58,5 +58,5 @@
             <geometry>
                 <mesh
-                    filename="package://turtlebot3_common/meshes/burger_base.dae"
+                    filename="package://armmy_turtlebot3/models/turtlebot3_common/meshes/burger_base.dae"
                     scale="0.001 0.001 0.001" />
             </geometry>
@@ -85,5 +85,5 @@
             <geometry>
                 <mesh
-                    filename="package://turtlebot3_common/meshes/tire.dae"
+                    filename="package://armmy_turtlebot3/models/turtlebot3_common/meshes/tire.dae"
                     scale="0.001 0.001 0.001" />
             </geometry>
@@ -112,5 +112,5 @@
             <geometry>
                 <mesh
-                    filename="package://turtlebot3_common/meshes/tire.dae"
+                    filename="package://armmy_turtlebot3/models/turtlebot3_common/meshes/tire.dae"
                     scale="0.001 0.001 0.001" />
             </geometry>
