Commit message: add omni robot

File: armmy_turtlebot3/urdf/tb3_custom/arm.xacro (robot description, xacro)
@@ -17,5 +17,5 @@
         </collision>
         <inertial>
-            <mass value="0.1" />
+            <mass value="0.02" />
             <inertia ixx="0.001" ixy="0" ixz="0" iyy="0.001" iyz="0" izz="0.001" />
         </inertial>
