Commit message: finish omni velocity control

File: armmy_omnibot/robots/omni_robot.urdf.xacro (robot description, xacro)
@@ -53,9 +53,117 @@
   </xacro:roller_v0>
   <!-- 2nd wheel -->
+  <xacro:wheel_v0 prefix="second" parent="base_link">
+    <origin xyz="-0.038375 0.0 -0.0" rpy="0 0 ${M_PI/2}" />
+    <axis xyz="0.0 1.0 0.0" />
+  </xacro:wheel_v0>
+  <xacro:roller_v0 prefix="r1_S" parent="second_wheel_link">
+    <origin xyz="0.01275 0.004625 -0.00925" rpy="0 0 0" />
+    <axis xyz="0.0 0.0 -1.0" />
+  </xacro:roller_v0>
+  <xacro:roller_v0 prefix="r2_S" parent="second_wheel_link">
+    <origin xyz="-0.00925 0.004625 -0.01275" rpy="0 ${M_PI/2} 0" />
+    <axis xyz="0.0 0.0 -1.0" />
+  </xacro:roller_v0>
+  <xacro:roller_v0 prefix="r3_S" parent="second_wheel_link">
+    <origin xyz="-0.01275 0.004625 0.00925" rpy="0 ${M_PI} 0" />
+    <axis xyz="0.0 0.0 -1.0" />
+  </xacro:roller_v0>
+  <xacro:roller_v0 prefix="r4_S" parent="second_wheel_link">
+    <origin xyz="0.00925 0.004625 0.01275" rpy="0 ${3*M_PI/2} 0" />
+    <axis xyz="0.0 0.0 -1.0" />
+  </xacro:roller_v0>
+  <xacro:roller_v0 prefix="r5_S" parent="second_wheel_link">
+    <origin xyz="0.015556 0.013875 -0.002475" rpy="0 ${-3*M_PI/4} 0" />
+    <axis xyz="0.0 0.0 -1.0" />
+  </xacro:roller_v0>
+  <xacro:roller_v0 prefix="r6_S" parent="second_wheel_link">
+    <origin xyz="-0.002475 0.013875 -0.015556" rpy="0 ${-M_PI/4} 0" />
+    <axis xyz="0.0 0.0 -1.0" />
+  </xacro:roller_v0>
+  <xacro:roller_v0 prefix="r7_S" parent="second_wheel_link">
+    <origin xyz="-0.015556 0.013875 0.002475" rpy="0 ${M_PI/4} 0" />
+    <axis xyz="0.0 0.0 -1.0" />
+  </xacro:roller_v0>
+  <xacro:roller_v0 prefix="r8_S" parent="second_wheel_link">
+    <origin xyz="0.002475 0.013875 0.015556" rpy="0 ${-5*M_PI/4} 0" />
+    <axis xyz="0.0 0.0 -1.0" />
+  </xacro:roller_v0>
   <!-- 3rd wheel -->
+  <xacro:wheel_v0 prefix="third" parent="base_link">
+    <origin xyz="-0.0 -0.038375 -0.0" rpy="0 0 ${M_PI}" />
+    <axis xyz="0.0 1.0 0.0" />
+  </xacro:wheel_v0>
+  <xacro:roller_v0 prefix="r1_T" parent="third_wheel_link">
+    <origin xyz="0.01275 0.004625 -0.00925" rpy="0 0 0" />
+    <axis xyz="0.0 0.0 -1.0" />
+  </xacro:roller_v0>
+  <xacro:roller_v0 prefix="r2_T" parent="third_wheel_link">
+    <origin xyz="-0.00925 0.004625 -0.01275" rpy="0 ${M_PI/2} 0" />
+    <axis xyz="0.0 0.0 -1.0" />
+  </xacro:roller_v0>
+  <xacro:roller_v0 prefix="r3_T" parent="third_wheel_link">
+    <origin xyz="-0.01275 0.004625 0.00925" rpy="0 ${M_PI} 0" />
+    <axis xyz="0.0 0.0 -1.0" />
+  </xacro:roller_v0>
+  <xacro:roller_v0 prefix="r4_T" parent="third_wheel_link">
+    <origin xyz="0.00925 0.004625 0.01275" rpy="0 ${3*M_PI/2} 0" />
+    <axis xyz="0.0 0.0 -1.0" />
+  </xacro:roller_v0>
+  <xacro:roller_v0 prefix="r5_T" parent="third_wheel_link">
+    <origin xyz="0.015556 0.013875 -0.002475" rpy="0 ${-3*M_PI/4} 0" />
+    <axis xyz="0.0 0.0 -1.0" />
+  </xacro:roller_v0>
+  <xacro:roller_v0 prefix="r6_T" parent="third_wheel_link">
+    <origin xyz="-0.002475 0.013875 -0.015556" rpy="0 ${-M_PI/4} 0" />
+    <axis xyz="0.0 0.0 -1.0" />
+  </xacro:roller_v0>
+  <xacro:roller_v0 prefix="r7_T" parent="third_wheel_link">
+    <origin xyz="-0.015556 0.013875 0.002475" rpy="0 ${M_PI/4} 0" />
+    <axis xyz="0.0 0.0 -1.0" />
+  </xacro:roller_v0>
+  <xacro:roller_v0 prefix="r8_T" parent="third_wheel_link">
+    <origin xyz="0.002475 0.013875 0.015556" rpy="0 ${-5*M_PI/4} 0" />
+    <axis xyz="0.0 0.0 -1.0" />
+  </xacro:roller_v0>
   <!-- 4th wheel -->
+  <xacro:wheel_v0 prefix="fourth" parent="base_link">
+    <origin xyz="0.038375 0.0 -0.0" rpy="0 0 ${3*M_PI/2}" />
+    <axis xyz="0.0 1.0 0.0" />
+  </xacro:wheel_v0>
+  <xacro:roller_v0 prefix="r1_R" parent="fourth_wheel_link">
+    <origin xyz="0.01275 0.004625 -0.00925" rpy="0 0 0" />
+    <axis xyz="0.0 0.0 -1.0" />
+  </xacro:roller_v0>
+  <xacro:roller_v0 prefix="r2_R" parent="fourth_wheel_link">
+    <origin xyz="-0.00925 0.004625 -0.01275" rpy="0 ${M_PI/2} 0" />
+    <axis xyz="0.0 0.0 -1.0" />
+  </xacro:roller_v0>
+  <xacro:roller_v0 prefix="r3_R" parent="fourth_wheel_link">
+    <origin xyz="-0.01275 0.004625 0.00925" rpy="0 ${M_PI} 0" />
+    <axis xyz="0.0 0.0 -1.0" />
+  </xacro:roller_v0>
+  <xacro:roller_v0 prefix="r4_R" parent="fourth_wheel_link">
+    <origin xyz="0.00925 0.004625 0.01275" rpy="0 ${3*M_PI/2} 0" />
+    <axis xyz="0.0 0.0 -1.0" />
+  </xacro:roller_v0>
+  <xacro:roller_v0 prefix="r5_R" parent="fourth_wheel_link">
+    <origin xyz="0.015556 0.013875 -0.002475" rpy="0 ${-3*M_PI/4} 0" />
+    <axis xyz="0.0 0.0 -1.0" />
+  </xacro:roller_v0>
+  <xacro:roller_v0 prefix="r6_R" parent="fourth_wheel_link">
+    <origin xyz="-0.002475 0.013875 -0.015556" rpy="0 ${-M_PI/4} 0" />
+    <axis xyz="0.0 0.0 -1.0" />
+  </xacro:roller_v0>
+  <xacro:roller_v0 prefix="r7_R" parent="fourth_wheel_link">
+    <origin xyz="-0.015556 0.013875 0.002475" rpy="0 ${M_PI/4} 0" />
+    <axis xyz="0.0 0.0 -1.0" />
+  </xacro:roller_v0>
+  <xacro:roller_v0 prefix="r8_R" parent="fourth_wheel_link">
+    <origin xyz="0.002475 0.013875 0.015556" rpy="0 ${-5*M_PI/4} 0" />
+    <axis xyz="0.0 0.0 -1.0" />
+  </xacro:roller_v0>
   <!-- lidar sensor -->
   <xacro:lidar_v0 prefix="front" parent="base_link">
-    <origin xyz="0 0 0.1395" />
+    <origin xyz="0 0 0.005000000000000001" />
   </xacro:lidar_v0>
   <!-- ===============  Transmission =============== -->
@@ -88,4 +196,5 @@
       </command_interface>
       <state_interface name="velocity" />
+      <state_interface name="position" />
     </joint>
     <joint name="second_wheel_joint">
@@ -95,4 +204,5 @@
       </command_interface>
       <state_interface name="velocity" />
+      <state_interface name="position" />
     </joint>
     <joint name="third_wheel_joint">
@@ -102,4 +212,5 @@
       </command_interface>
       <state_interface name="velocity" />
+      <state_interface name="position" />
     </joint>
     <joint name="fourth_wheel_joint">
@@ -109,10 +220,10 @@
       </command_interface>
       <state_interface name="velocity" />
+      <state_interface name="position" />
     </joint>
   </ros2_control>
   <gazebo>
     <plugin name="gazebo_ros2_control" filename="libgazebo_ros2_control.so">
-      <parameters>
-        /home/armmy2530/Documents/ros2/EIC_Turtlebot3/src/omni_navigation/src/gazebo_simulation/models/rs_robot/config/controllers.yaml</parameters>
+      <parameters>$(find armmy_omnibot)/config/ros2_controller/my_controllers.yaml</parameters>
     </plugin>
   </gazebo>

File: armmy_omnibot/urdf/lidar/lidar.gazebo.xacro (robot description, xacro)
@@ -1,36 +1,45 @@
 <?xml version="1.0"?>
 <robot xmlns:xacro="http://ros.org/wiki/xacro">
-  <xacro:macro name="lidar_gazebo_v0" params="prefix min_rad max_rad min_range max_range">
-	<gazebo reference="${prefix}_lidar_link">
-      <sensor type="ray" name="${prefix}_lidar_sensor">
-		<pose>0 0 0 0 0 0</pose>
-		<visualize>true</visualize>
-		<update_rate>40</update_rate>
-		<ray>
-          <scan>
-	    <horizontal>
-              <samples>720</samples>
-              <resolution>1</resolution>
-              <min_angle>${min_rad}</min_angle>
-              <max_angle>${max_rad}</max_angle>
-	    </horizontal>
-          </scan>
-          <range>
-		<min>${min_range}</min>
-		<max>${max_range}</max>
-		<resolution>0.01</resolution>
-          </range>
-          <noise>
-		<type>gaussian</type>
-		<mean>0.0</mean>
-		<stddev>0.03</stddev>
-          </noise>
-		</ray>
-		<plugin name="gazebo_ros_${prefix}_lidar_controller" filename="libgazebo_ros_laser.so">
-          <topicName>${prefix}/scan</topicName> <!-- do ont set it to base_scan -->
+	<xacro:macro name="lidar_gazebo_v0" params="prefix min_rad max_rad min_range max_range">
+		<gazebo reference="${prefix}_lidar_link">
+			<sensor type="ray" name="${prefix}_lidar_sensor">
+				<pose>0 0 0 0 0 0</pose>
+				<visualize>true</visualize>
+				<update_rate>40</update_rate>
+				<ray>
+					<scan>
+						<horizontal>
+							<samples>720</samples>
+							<resolution>1</resolution>
+							<min_angle>${min_rad}</min_angle>
+							<max_angle>${max_rad}</max_angle>
+						</horizontal>
+					</scan>
+					<range>
+						<min>${min_range}</min>
+						<max>${max_range}</max>
+						<resolution>0.01</resolution>
+					</range>
+					<noise>
+						<type>gaussian</type>
+						<mean>0.0</mean>
+						<stddev>0.01</stddev>
+					</noise>
+				</ray>
+				<plugin name="turtlebot3_laserscan" filename="libgazebo_ros_ray_sensor.so">
+					<ros>
+						<!-- <namespace>/tb3</namespace> -->
+						<remapping>~/out:=scan</remapping>
+					</ros>
+					<output_type>sensor_msgs/LaserScan</output_type>
+					<frame_name>${prefix}_lidar_link</frame_name>
+				</plugin>
+				<!-- <plugin name="gazebo_ros_${prefix}_lidar_controller"
+				filename="libgazebo_ros_laser.so">
+          <topicName>${prefix}/scan</topicName>
           <frameName>${prefix}_lidar_link</frameName>
-		</plugin>
-      </sensor>
-	</gazebo>
-  </xacro:macro>
+		</plugin> -->
+			</sensor>
+		</gazebo>
+	</xacro:macro>
 </robot>

File: armmy_omnibot/urdf/roller/roller.urdf.xacro (robot description, xacro)
@@ -23,5 +23,5 @@
       <inertial>
         <origin xyz="0.0 0.0 0.0" />
-        <mass value="0.009" />
+        <mass value="0.02" />
         <inertia ixx="0.000001257" ixy="0" ixz="0" iyy="0.000000342" iyz="0" izz="0.000001257" />
       </inertial>

Commit message: add angular velocity mesurement (something wrong)

File: armmy_omnibot/robots/omni_robot.urdf.xacro (robot description, xacro)
@@ -12,5 +12,5 @@
   <link name="base_footprint" />
   <xacro:base_v0 parent="base_footprint">
-    <origin xyz="0 0 0" rpy="0 0 0" />
+    <origin xyz="0 0 0" rpy="0 0 ${M_PI / 4}" />
   </xacro:base_v0>
   <!-- Wheel -->
