Commit message: finish 3 wheel fk

File: armmy_omnibot/robots/3wheel_omni_robot.urdf.xacro (robot description, xacro)
@@ -8,4 +8,5 @@
   <xacro:include filename="$(find armmy_omnibot)/urdf/roller/roller.urdf.xacro" />
   <xacro:include filename="$(find armmy_omnibot)/urdf/lidar/lidar.urdf.xacro" />
+  <xacro:include filename="$(find armmy_omnibot)/urdf/color.xacro" />
   <!-- =============== Link & Joint =============== -->
   <!-- Base -->
@@ -17,5 +18,5 @@
   <!-- 1st wheel -->
   <xacro:wheel_v0 prefix="first" parent="base_link">
-    <origin xyz="-0.0 0.038375 -0.0" rpy="0 0 0" />
+    <origin xyz="-0.038375 0.0 -0.0" rpy="0 0 ${M_PI/2}" />
     <axis xyz="0.0 1.0 0.0" />
   </xacro:wheel_v0>
@@ -54,5 +55,5 @@
   <!-- 2nd wheel -->
   <xacro:wheel_v0 prefix="second" parent="base_link">
-    <origin xyz="-0.03323372487 -0.0191875 -0.0" rpy="0 0 ${4*M_PI/6}" />
+    <origin xyz="0.0191875 -0.03323372487 -0.0" rpy="0 0 ${7*M_PI/6}" />
     <axis xyz="0.0 1.0 0.0" />
   </xacro:wheel_v0>
@@ -91,5 +92,5 @@
   <!-- 3rd wheel -->
   <xacro:wheel_v0 prefix="third" parent="base_link">
-    <origin xyz="0.03323372487 -0.0191875 -0.0" rpy="0 0 ${8*M_PI/6}" />
+    <origin xyz="0.0191875 0.03323372487 -0.0" rpy="0 0 ${11*M_PI/6}" />
     <axis xyz="0.0 1.0 0.0" />
   </xacro:wheel_v0>
@@ -178,5 +179,5 @@
   <gazebo>
     <plugin name="gazebo_ros2_control" filename="libgazebo_ros2_control.so">
-      <parameters>$(find armmy_omnibot)/config/ros2_controller/my_controllers.yaml</parameters>
+      <parameters>$(find armmy_omnibot)/config/ros2_controller/3wheel_controllers.yaml</parameters>
     </plugin>
     <plugin name="gazebo_ros_p3d" filename="libgazebo_ros_p3d.so">

File: armmy_omnibot/robots/omni_robot.urdf.xacro (robot description, xacro)
@@ -8,4 +8,5 @@
   <xacro:include filename="$(find armmy_omnibot)/urdf/roller/roller.urdf.xacro" />
   <xacro:include filename="$(find armmy_omnibot)/urdf/lidar/lidar.urdf.xacro" />
+  <xacro:include filename="$(find armmy_omnibot)/urdf/color.xacro" />
   <!-- =============== Link & Joint =============== -->
   <!-- Base -->

File: armmy_omnibot/urdf/base/base.urdf.xacro (robot description, xacro)
@@ -18,4 +18,5 @@
             scale="0.001 0.001 0.001" />
         </geometry>
+        <material name="white" />
       </visual>
       <collision>

File: armmy_omnibot/urdf/omni_wheel/omni_wheel.urdf.xacro (robot description, xacro)
@@ -1,6 +1,6 @@
 <?xml version="1.0"?>
 <robot xmlns:xacro="http://ros.org/wiki/xacro">
-  <xacro:include filename="$(find armmy_omnibot)/urdf/omni_wheel/omni_wheel.transmission.xacro"/>
-  <xacro:include filename="$(find armmy_omnibot)/urdf/omni_wheel/omni_wheel.gazebo.xacro"/>
+  <xacro:include filename="$(find armmy_omnibot)/urdf/omni_wheel/omni_wheel.transmission.xacro" />
+  <xacro:include filename="$(find armmy_omnibot)/urdf/omni_wheel/omni_wheel.gazebo.xacro" />
   <xacro:include filename="$(find armmy_omnibot)/urdf/inertial_macros.xacro" />
   <xacro:property name="wheel_thickness" value="0.0185" />
@@ -8,51 +8,54 @@
   <xacro:property name="wheel_mass" value="0.05" />
   <xacro:macro name="wheel_v0" params="prefix parent *joint_origin *joint_axis">
-	<joint name="${prefix}_wheel_joint" type="continuous">
-	  <xacro:insert_block name="joint_origin"/>
-	  <parent link="${parent}"/>
-	  <child link="${prefix}_wheel_link"/>
-          <limit effort="100" velocity="100"/>
-	  <xacro:insert_block name="joint_axis"/>
-	</joint>
-	<link name="${prefix}_wheel_link">
-	  <visual>
-		<geometry>
-          <mesh filename="package://armmy_omnibot/meshes/omni_wheel/wheel_base.stl" scale="0.001 0.001 0.001" />
-		</geometry>
-	  </visual>
-	  <collision>
-		<geometry>
-          <mesh filename="package://armmy_omnibot/meshes/omni_wheel/wheel_base.stl" scale="0.001 0.001 0.001" />
-		</geometry>
-	  </collision>
-    <xacro:inertial_cylinder mass="${wheel_mass}" length="${wheel_thickness}"
+    <joint name="${prefix}_wheel_joint" type="continuous">
+      <xacro:insert_block name="joint_origin" />
+      <parent link="${parent}" />
+      <child link="${prefix}_wheel_link" />
+      <limit effort="100" velocity="100" />
+      <xacro:insert_block name="joint_axis" />
+    </joint>
+    <link name="${prefix}_wheel_link">
+      <visual>
+        <geometry>
+          <mesh filename="package://armmy_omnibot/meshes/omni_wheel/wheel_base.stl"
+            scale="0.001 0.001 0.001" />
+        </geometry>
+        <material name="light_black" />
+      </visual>
+      <collision>
+        <geometry>
+          <mesh filename="package://armmy_omnibot/meshes/omni_wheel/wheel_base.stl"
+            scale="0.001 0.001 0.001" />
+        </geometry>
+      </collision>
+      <xacro:inertial_cylinder mass="${wheel_mass}" length="${wheel_thickness}"
         radius="${wheel_radian}">
         <origin xyz="0 ${wheel_thickness/2} 0" rpy="1.570796327 0 0" />
       </xacro:inertial_cylinder>
-	  <!-- <inertial>
+      <!-- <inertial>
 		<origin xyz="0.0 -0.0 -0.0"/>
 		<mass value="0.25"/>
 		<inertia ixx="0.00031" ixy="0" ixz="0" iyy="0.0005" iyz="0" izz="0.00031"/>
 	  </inertial> -->
-          <surface>
-            <friction>
-              <ode>
-                <mu1>1.2</mu1>
-                <mu2>1.2</mu2>
-                <kp>1e15</kp>
-                <kd>1e13</kd>
-              </ode>
-            </friction>
-            <bounce>
-              <restitution_coefficient>0.01</restitution_coefficient>
-              <threshold>0</threshold>
-            </bounce>
-            <contact>
-              <ode>
-                <max_vel>10</max_vel>
-              </ode>
-            </contact>
-          </surface>
-	</link>
+      <surface>
+        <friction>
+          <ode>
+            <mu1>1.2</mu1>
+            <mu2>1.2</mu2>
+            <kp>1e15</kp>
+            <kd>1e13</kd>
+          </ode>
+        </friction>
+        <bounce>
+          <restitution_coefficient>0.01</restitution_coefficient>
+          <threshold>0</threshold>
+        </bounce>
+        <contact>
+          <ode>
+            <max_vel>10</max_vel>
+          </ode>
+        </contact>
+      </surface>
+    </link>
   </xacro:macro>
 </robot>

File: armmy_omnibot/urdf/roller/roller.urdf.xacro (robot description, xacro)
@@ -20,4 +20,5 @@
             scale="0.001 0.001 0.001" />
         </geometry>
+        <material name="black" />
       </visual>
       <collision>
