Commit message: need to fix slow sim in new gz (too much collision of roller wheel)

File: armmy_omnibot/robots/newgz_omni_robot.urdf.xacro (robot description, xacro)
@@ -187,7 +187,7 @@
   <xacro:lidar_gazebo_v0 prefix="front" min_rad="-3.14" max_rad="3.14" min_range="0.1"
     max_range="10" />
-  <ros2_control name="IgnitionSystem" type="system">
+  <ros2_control name="GazeboSystem" type="system">
     <hardware>
-      <plugin>ign_ros2_control/IgnitionSystem</plugin>
+      <plugin>gz_ros2_control/GazeboSimSystem</plugin>
     </hardware>
     <joint name="first_wheel_joint">
@@ -225,5 +225,6 @@
   </ros2_control>
   <gazebo>
-    <plugin name="ign_ros2_control::IgnitionROS2ControlPlugin" filename="libign_ros2_control-system.so">
+    <plugin name="gz_ros2_control::GazeboSimROS2ControlPlugin"
+      filename="libgz_ros2_control-system.so">
       <parameters>$(find armmy_omnibot)/config/ros2_controller/my_controllers.yaml</parameters>
     </plugin>

File: armmy_omnibot/urdf/lidar/lidar_gz.urdf.xacro (robot description, xacro)
@@ -11,3 +11,34 @@
 	</link>
   </xacro:macro>
+  <xacro:macro name="lidar_gazebo_v0" params="prefix min_rad max_rad min_range max_range">
+	<gazebo reference="${prefix}_lidar_link">
+        <sensor name="laser" type="gpu_lidar">
+            <visualize>false</visualize>
+            <pose>0 0 0 0 0 0</pose>
+            <update_rate>5</update_rate>
+            <lidar>
+                <scan>
+                    <horizontal>
+                        <samples>360</samples>
+                        <resolution>1.000000</resolution>
+                        <min_angle>${min_rad}</min_angle>
+                        <max_angle>${max_rad}</max_angle>
+                    </horizontal>
+                </scan>
+                <range>
+                    <min>${min_range}</min>
+                    <max>${max_range}</max>
+                    <resolution>0.015000</resolution>
+                </range>
+                <noise>
+                    <type>gaussian</type>
+                    <mean>0.0</mean>
+                    <stddev>0.01</stddev>
+                </noise>
+            </lidar>
+            <topic>scan</topic>
+            <gz_frame_id>${prefix}_lidar_link</gz_frame_id>
+        </sensor>
+    </gazebo>
+  </xacro:macro>
 </robot>

File: armmy_omnibot/urdf/omni_wheel/omni_wheel.urdf.xacro (robot description, xacro)
@@ -23,19 +23,14 @@
         <material name="light_black" />
       </visual>
-      <collision>
+      <!-- <collision>
         <geometry>
           <mesh filename="package://armmy_omnibot/meshes/omni_wheel/wheel_base.stl"
             scale="0.001 0.001 0.001" />
         </geometry>
-      </collision>
+      </collision> -->
       <xacro:inertial_cylinder mass="${wheel_mass}" length="${wheel_thickness}"
         radius="${wheel_radian}">
         <origin xyz="0 ${wheel_thickness/2} 0" rpy="1.570796327 0 0" />
       </xacro:inertial_cylinder>
-      <!-- <inertial>
-		<origin xyz="0.0 -0.0 -0.0"/>
-		<mass value="0.25"/>
-		<inertia ixx="0.00031" ixy="0" ixz="0" iyy="0.0005" iyz="0" izz="0.00031"/>
-	  </inertial> -->
       <surface>
         <friction>

File: armmy_turtlebot3/urdf/tb3_custom_newgz/ros2_control.xacro (robot description, xacro)
@@ -18,6 +18,6 @@
                     <param name="max">10</param>
                 </command_interface>
-                <state_interface name="velocity"/>
-                <state_interface name="position"/>
+                <state_interface name="velocity" />
+                <state_interface name="position" />
             </joint>
             <joint name="wheel_right_joint">
@@ -26,13 +26,13 @@
                     <param name="max">10</param>
                 </command_interface>
-                <state_interface name="velocity"/>
-                <state_interface name="position"/>
+                <state_interface name="velocity" />
+                <state_interface name="position" />
             </joint>
         </ros2_control>
     </xacro:unless>
     <xacro:if value="$(arg sim_mode)">
-        <ros2_control name="IgnitionSystem" type="system">
+        <ros2_control name="GazeboSystem" type="system">
             <hardware>
-                <plugin>ign_ros2_control/IgnitionSystem</plugin>
+                <plugin>gz_ros2_control/GazeboSimSystem</plugin>
             </hardware>
             <joint name="wheel_left_joint">
@@ -41,6 +41,6 @@
                     <param name="max">10</param>
                 </command_interface>
-                <state_interface name="velocity"/>
-                <state_interface name="position"/>
+                <state_interface name="velocity" />
+                <state_interface name="position" />
             </joint>
             <joint name="wheel_right_joint">
@@ -49,18 +49,19 @@
                     <param name="max">10</param>
                 </command_interface>
-                <state_interface name="velocity"/>
-                <state_interface name="position"/>
+                <state_interface name="velocity" />
+                <state_interface name="position" />
             </joint>
             <joint name="arm_joint">
-                <command_interface name="position"/>
+                <command_interface name="position" />
                 <state_interface name="position">
-                  <param name="initial_value">0.0</param>
+                    <param name="initial_value">0.0</param>
                 </state_interface>
-                <state_interface name="velocity"/>
+                <state_interface name="velocity" />
             </joint>
         </ros2_control>
     </xacro:if>
     <gazebo>
-        <plugin name="ign_ros2_control::IgnitionROS2ControlPlugin" filename="libign_ros2_control-system.so">
+        <plugin name="gz_ros2_control::GazeboSimROS2ControlPlugin"
+            filename="libgz_ros2_control-system.so">
             <parameters>$(find armmy_turtlebot3)/config/ros2_controller/my_controllers.yaml</parameters>
             <parameters>$(find armmy_turtlebot3)/config/ros2_controller/gaz_ros2_ctl_use_sim.yaml</parameters>

Commit message: add imu

File: armmy_omnibot/robots/newgz_omni_robot.urdf.xacro (robot description, xacro)
@@ -4,9 +4,10 @@
   <xacro:arg name="use_ros2_control" default="true" />
   <xacro:arg name="sim_mode" default="false" />
-  <xacro:include filename="$(find armmy_omnibot)/urdf/base/base.urdf.xacro" />
-  <xacro:include filename="$(find armmy_omnibot)/urdf/omni_wheel/omni_wheel.urdf.xacro" />
-  <xacro:include filename="$(find armmy_omnibot)/urdf/roller/roller.urdf.xacro" />
-  <xacro:include filename="$(find armmy_omnibot)/urdf/lidar/lidar_gz.urdf.xacro" />
-  <xacro:include filename="$(find armmy_omnibot)/urdf/color.xacro" />
+  <xacro:include filename="$(find armmy_omnibot)/urdf/base/base.urdf.xacro"/>
+  <xacro:include filename="$(find armmy_omnibot)/urdf/omni_wheel/omni_wheel.urdf.xacro"/>
+  <xacro:include filename="$(find armmy_omnibot)/urdf/roller/roller.urdf.xacro"/>
+  <xacro:include filename="$(find armmy_omnibot)/urdf/lidar/lidar_gz.urdf.xacro"/>
+  <xacro:include filename="$(find armmy_omnibot)/urdf/imu/imu_gz.urdf.xacro"/>
+  <xacro:include filename="$(find armmy_omnibot)/urdf/color.xacro"/>
   <!-- =============== Link & Joint =============== -->
   <!-- Base -->
@@ -166,6 +167,12 @@
   <!-- lidar sensor -->
   <xacro:lidar_v0 prefix="top" parent="base_link">
-    <origin xyz="0 0 0.005000000000000001" />
+    <origin xyz="0 0 0.05000000000000001" />
   </xacro:lidar_v0>
+  <xacro:lidar_gazebo_v0 prefix="top" min_rad="-3.14" max_rad="3.14" min_range="0.02" max_range="10" />
+  <!-- imu sensor -->
+  <xacro:imu_v0 prefix="top" parent="base_link">
+    <origin xyz="0 0 0.05000000000000001" />
+  </xacro:imu_v0>
+  <xacro:imu_gazebo_v0 prefix="top" />
   <!-- ===============  Transmission =============== -->
   <xacro:wheel_trans_v0 prefix="first" />
@@ -173,8 +180,4 @@
   <xacro:wheel_trans_v0 prefix="third" />
   <xacro:wheel_trans_v0 prefix="fourth" />
-  <!-- =============== Gazebo =============== -->
-  <!-- <gazebo>
-    <plugin name="gazebo_ros_control" filename="libgazebo_ros_control.so" />
-  </gazebo> -->
   <!-- Base -->
   <xacro:base_gazebo_v0 />
@@ -184,7 +187,4 @@
   <xacro:wheel_gazebo_v0 prefix="third" />
   <xacro:wheel_gazebo_v0 prefix="fourth" />
-  <!-- lidar sensor -->
-  <xacro:lidar_gazebo_v0 prefix="front" min_rad="-3.14" max_rad="3.14" min_range="0.1"
-    max_range="10" />
   <ros2_control name="GazeboSystem" type="system">
     <hardware>

File: armmy_omnibot/urdf/lidar/lidar.gz.xacro (robot description, xacro)
@@ -3,8 +3,8 @@
 	<xacro:macro name="lidar_gazebo_v0" params="prefix min_rad max_rad min_range max_range">
 		<gazebo reference="${prefix}_lidar_link">
-			<sensor name="${prefix}_lidar_sensor" type="gpu_lidar">
+			<sensor name="laser" type="gpu_lidar">
 				<visualize>false</visualize>
 				<pose>0 0 0 0 0 0</pose>
-				<update_rate>5</update_rate>
+				<update_rate>40</update_rate>
 				<lidar>
 					<scan>
@@ -12,11 +12,11 @@
 							<samples>360</samples>
 							<resolution>1.000000</resolution>
-							<min_angle>0.000000</min_angle>
-							<max_angle>6.280000</max_angle>
+							<min_angle>${min_rad}</min_angle>
+							<max_angle>${max_rad}</max_angle>
 						</horizontal>
 					</scan>
 					<range>
-						<min>0.120000</min>
-						<max>3.5</max>
+						<min>${min_range}</min>
+						<max>${max_range}</max>
 						<resolution>0.015000</resolution>
 					</range>

File: armmy_omnibot/urdf/lidar/lidar_gz.urdf.xacro (robot description, xacro)
@@ -1,44 +1,13 @@
 <?xml version="1.0"?>
 <robot xmlns:xacro="http://ros.org/wiki/xacro">
-  <xacro:include filename="$(find armmy_omnibot)/urdf/lidar/lidar.gz.xacro"/>
+  <xacro:include filename="$(find armmy_omnibot)/urdf/lidar/lidar.gz.xacro" />
   <xacro:macro name="lidar_v0" params="prefix parent *joint_origin">
-	<joint name="${prefix}_lidar_joint" type="fixed">
-	  <xacro:insert_block name="joint_origin"/>
-	  <parent link="${parent}"/>
-	  <child link="${prefix}_lidar_link"/>
-	</joint>
-	<link name="${prefix}_lidar_link">
-	</link>
-  </xacro:macro>
-  <xacro:macro name="lidar_gazebo_v0" params="prefix min_rad max_rad min_range max_range">
-	<gazebo reference="${prefix}_lidar_link">
-        <sensor name="laser" type="gpu_lidar">
-            <visualize>false</visualize>
-            <pose>0 0 0 0 0 0</pose>
-            <update_rate>5</update_rate>
-            <lidar>
-                <scan>
-                    <horizontal>
-                        <samples>360</samples>
-                        <resolution>1.000000</resolution>
-                        <min_angle>${min_rad}</min_angle>
-                        <max_angle>${max_rad}</max_angle>
-                    </horizontal>
-                </scan>
-                <range>
-                    <min>${min_range}</min>
-                    <max>${max_range}</max>
-                    <resolution>0.015000</resolution>
-                </range>
-                <noise>
-                    <type>gaussian</type>
-                    <mean>0.0</mean>
-                    <stddev>0.01</stddev>
-                </noise>
-            </lidar>
-            <topic>scan</topic>
-            <gz_frame_id>${prefix}_lidar_link</gz_frame_id>
-        </sensor>
-    </gazebo>
+    <joint name="${prefix}_lidar_joint" type="fixed">
+      <xacro:insert_block name="joint_origin" />
+      <parent link="${parent}" />
+      <child link="${prefix}_lidar_link" />
+    </joint>
+    <link name="${prefix}_lidar_link">
+    </link>
   </xacro:macro>
 </robot>

Commit message: changing omni collision in new gz

File: armmy_omnibot/robots/newgz_omni_robot.urdf.xacro (robot description, xacro)
@@ -5,6 +5,5 @@
   <xacro:arg name="sim_mode" default="false" />
   <xacro:include filename="$(find armmy_omnibot)/urdf/base/base.urdf.xacro"/>
-  <xacro:include filename="$(find armmy_omnibot)/urdf/omni_wheel/omni_wheel.urdf.xacro"/>
-  <xacro:include filename="$(find armmy_omnibot)/urdf/roller/roller.urdf.xacro"/>
+  <xacro:include filename="$(find armmy_omnibot)/urdf/omni_wheel/gz_omni_wheel.urdf.xacro"/>
   <xacro:include filename="$(find armmy_omnibot)/urdf/lidar/lidar_gz.urdf.xacro"/>
   <xacro:include filename="$(find armmy_omnibot)/urdf/imu/imu_gz.urdf.xacro"/>
@@ -22,36 +21,4 @@
     <axis xyz="0.0 1.0 0.0" />
   </xacro:wheel_v0>
-  <xacro:roller_v0 prefix="r1_F" parent="first_wheel_link">
-    <origin xyz="0.01275 0.004625 -0.00925" rpy="0 0 0" />
-    <axis xyz="0.0 0.0 -1.0" />
-  </xacro:roller_v0>
-  <xacro:roller_v0 prefix="r2_F" parent="first_wheel_link">
-    <origin xyz="-0.00925 0.004625 -0.01275" rpy="0 ${M_PI/2} 0" />
-    <axis xyz="0.0 0.0 -1.0" />
-  </xacro:roller_v0>
-  <xacro:roller_v0 prefix="r3_F" parent="first_wheel_link">
-    <origin xyz="-0.01275 0.004625 0.00925" rpy="0 ${M_PI} 0" />
-    <axis xyz="0.0 0.0 -1.0" />
-  </xacro:roller_v0>
-  <xacro:roller_v0 prefix="r4_F" parent="first_wheel_link">
-    <origin xyz="0.00925 0.004625 0.01275" rpy="0 ${3*M_PI/2} 0" />
-    <axis xyz="0.0 0.0 -1.0" />
-  </xacro:roller_v0>
-  <xacro:roller_v0 prefix="r5_F" parent="first_wheel_link">
-    <origin xyz="0.015556 0.013875 -0.002475" rpy="0 ${-3*M_PI/4} 0" />
-    <axis xyz="0.0 0.0 -1.0" />
-  </xacro:roller_v0>
-  <xacro:roller_v0 prefix="r6_F" parent="first_wheel_link">
-    <origin xyz="-0.002475 0.013875 -0.015556" rpy="0 ${-M_PI/4} 0" />
-    <axis xyz="0.0 0.0 -1.0" />
-  </xacro:roller_v0>
-  <xacro:roller_v0 prefix="r7_F" parent="first_wheel_link">
-    <origin xyz="-0.015556 0.013875 0.002475" rpy="0 ${M_PI/4} 0" />
-    <axis xyz="0.0 0.0 -1.0" />
-  </xacro:roller_v0>
-  <xacro:roller_v0 prefix="r8_F" parent="first_wheel_link">
-    <origin xyz="0.002475 0.013875 0.015556" rpy="0 ${-5*M_PI/4} 0" />
-    <axis xyz="0.0 0.0 -1.0" />
-  </xacro:roller_v0>
   <!-- 2nd wheel -->
   <xacro:wheel_v0 prefix="second" parent="base_link">
@@ -59,36 +26,4 @@
     <axis xyz="0.0 1.0 0.0" />
   </xacro:wheel_v0>
-  <xacro:roller_v0 prefix="r1_S" parent="second_wheel_link">
-    <origin xyz="0.01275 0.004625 -0.00925" rpy="0 0 0" />
-    <axis xyz="0.0 0.0 -1.0" />
-  </xacro:roller_v0>
-  <xacro:roller_v0 prefix="r2_S" parent="second_wheel_link">
-    <origin xyz="-0.00925 0.004625 -0.01275" rpy="0 ${M_PI/2} 0" />
-    <axis xyz="0.0 0.0 -1.0" />
-  </xacro:roller_v0>
-  <xacro:roller_v0 prefix="r3_S" parent="second_wheel_link">
-    <origin xyz="-0.01275 0.004625 0.00925" rpy="0 ${M_PI} 0" />
-    <axis xyz="0.0 0.0 -1.0" />
-  </xacro:roller_v0>
-  <xacro:roller_v0 prefix="r4_S" parent="second_wheel_link">
-    <origin xyz="0.00925 0.004625 0.01275" rpy="0 ${3*M_PI/2} 0" />
-    <axis xyz="0.0 0.0 -1.0" />
-  </xacro:roller_v0>
-  <xacro:roller_v0 prefix="r5_S" parent="second_wheel_link">
-    <origin xyz="0.015556 0.013875 -0.002475" rpy="0 ${-3*M_PI/4} 0" />
-    <axis xyz="0.0 0.0 -1.0" />
-  </xacro:roller_v0>
-  <xacro:roller_v0 prefix="r6_S" parent="second_wheel_link">
-    <origin xyz="-0.002475 0.013875 -0.015556" rpy="0 ${-M_PI/4} 0" />
-    <axis xyz="0.0 0.0 -1.0" />
-  </xacro:roller_v0>
-  <xacro:roller_v0 prefix="r7_S" parent="second_wheel_link">
-    <origin xyz="-0.015556 0.013875 0.002475" rpy="0 ${M_PI/4} 0" />
-    <axis xyz="0.0 0.0 -1.0" />
-  </xacro:roller_v0>
-  <xacro:roller_v0 prefix="r8_S" parent="second_wheel_link">
-    <origin xyz="0.002475 0.013875 0.015556" rpy="0 ${-5*M_PI/4} 0" />
-    <axis xyz="0.0 0.0 -1.0" />
-  </xacro:roller_v0>
   <!-- 3rd wheel -->
   <xacro:wheel_v0 prefix="third" parent="base_link">
@@ -96,36 +31,4 @@
     <axis xyz="0.0 1.0 0.0" />
   </xacro:wheel_v0>
-  <xacro:roller_v0 prefix="r1_T" parent="third_wheel_link">
-    <origin xyz="0.01275 0.004625 -0.00925" rpy="0 0 0" />
-    <axis xyz="0.0 0.0 -1.0" />
-  </xacro:roller_v0>
-  <xacro:roller_v0 prefix="r2_T" parent="third_wheel_link">
-    <origin xyz="-0.00925 0.004625 -0.01275" rpy="0 ${M_PI/2} 0" />
-    <axis xyz="0.0 0.0 -1.0" />
-  </xacro:roller_v0>
-  <xacro:roller_v0 prefix="r3_T" parent="third_wheel_link">
-    <origin xyz="-0.01275 0.004625 0.00925" rpy="0 ${M_PI} 0" />
-    <axis xyz="0.0 0.0 -1.0" />
-  </xacro:roller_v0>
-  <xacro:roller_v0 prefix="r4_T" parent="third_wheel_link">
-    <origin xyz="0.00925 0.004625 0.01275" rpy="0 ${3*M_PI/2} 0" />
-    <axis xyz="0.0 0.0 -1.0" />
-  </xacro:roller_v0>
-  <xacro:roller_v0 prefix="r5_T" parent="third_wheel_link">
-    <origin xyz="0.015556 0.013875 -0.002475" rpy="0 ${-3*M_PI/4} 0" />
-    <axis xyz="0.0 0.0 -1.0" />
-  </xacro:roller_v0>
-  <xacro:roller_v0 prefix="r6_T" parent="third_wheel_link">
-    <origin xyz="-0.002475 0.013875 -0.015556" rpy="0 ${-M_PI/4} 0" />
-    <axis xyz="0.0 0.0 -1.0" />
-  </xacro:roller_v0>
-  <xacro:roller_v0 prefix="r7_T" parent="third_wheel_link">
-    <origin xyz="-0.015556 0.013875 0.002475" rpy="0 ${M_PI/4} 0" />
-    <axis xyz="0.0 0.0 -1.0" />
-  </xacro:roller_v0>
-  <xacro:roller_v0 prefix="r8_T" parent="third_wheel_link">
-    <origin xyz="0.002475 0.013875 0.015556" rpy="0 ${-5*M_PI/4} 0" />
-    <axis xyz="0.0 0.0 -1.0" />
-  </xacro:roller_v0>
   <!-- 4th wheel -->
   <xacro:wheel_v0 prefix="fourth" parent="base_link">
@@ -133,36 +36,4 @@
     <axis xyz="0.0 1.0 0.0" />
   </xacro:wheel_v0>
-  <xacro:roller_v0 prefix="r1_R" parent="fourth_wheel_link">
-    <origin xyz="0.01275 0.004625 -0.00925" rpy="0 0 0" />
-    <axis xyz="0.0 0.0 -1.0" />
-  </xacro:roller_v0>
-  <xacro:roller_v0 prefix="r2_R" parent="fourth_wheel_link">
-    <origin xyz="-0.00925 0.004625 -0.01275" rpy="0 ${M_PI/2} 0" />
-    <axis xyz="0.0 0.0 -1.0" />
-  </xacro:roller_v0>
-  <xacro:roller_v0 prefix="r3_R" parent="fourth_wheel_link">
-    <origin xyz="-0.01275 0.004625 0.00925" rpy="0 ${M_PI} 0" />
-    <axis xyz="0.0 0.0 -1.0" />
-  </xacro:roller_v0>
-  <xacro:roller_v0 prefix="r4_R" parent="fourth_wheel_link">
-    <origin xyz="0.00925 0.004625 0.01275" rpy="0 ${3*M_PI/2} 0" />
-    <axis xyz="0.0 0.0 -1.0" />
-  </xacro:roller_v0>
-  <xacro:roller_v0 prefix="r5_R" parent="fourth_wheel_link">
-    <origin xyz="0.015556 0.013875 -0.002475" rpy="0 ${-3*M_PI/4} 0" />
-    <axis xyz="0.0 0.0 -1.0" />
-  </xacro:roller_v0>
-  <xacro:roller_v0 prefix="r6_R" parent="fourth_wheel_link">
-    <origin xyz="-0.002475 0.013875 -0.015556" rpy="0 ${-M_PI/4} 0" />
-    <axis xyz="0.0 0.0 -1.0" />
-  </xacro:roller_v0>
-  <xacro:roller_v0 prefix="r7_R" parent="fourth_wheel_link">
-    <origin xyz="-0.015556 0.013875 0.002475" rpy="0 ${M_PI/4} 0" />
-    <axis xyz="0.0 0.0 -1.0" />
-  </xacro:roller_v0>
-  <xacro:roller_v0 prefix="r8_R" parent="fourth_wheel_link">
-    <origin xyz="0.002475 0.013875 0.015556" rpy="0 ${-5*M_PI/4} 0" />
-    <axis xyz="0.0 0.0 -1.0" />
-  </xacro:roller_v0>
   <!-- lidar sensor -->
   <xacro:lidar_v0 prefix="top" parent="base_link">

File: armmy_omnibot/urdf/omni_wheel/omni_wheel.urdf.xacro (robot description, xacro)
@@ -18,8 +18,8 @@
       <visual>
         <geometry>
-          <mesh filename="package://armmy_omnibot/meshes/omni_wheel/wheel_base.stl"
-            scale="0.001 0.001 0.001" />
+          <mesh filename="package://armmy_omnibot/meshes/omni_wheel/wheel_assembly.dae"
+            scale="1 1 1" />
         </geometry>
-        <material name="light_black" />
+        <!-- <material name="light_black" /> -->
       </visual>
       <!-- <collision>

File: armmy_omnibot/urdf/roller/roller.urdf.xacro (robot description, xacro)
@@ -3,4 +3,5 @@
   <xacro:property name="roller_length" value="0.0185" />
   <xacro:property name="roller_radius" value="0.00475" />
+  <xacro:property name="roller_tangent_radius" value="0.0175" />
   <xacro:property name="roller_mass" value="0.005" />
   <xacro:include filename="$(find armmy_omnibot)/urdf/roller/roller.transmission.xacro" />
@@ -23,13 +24,13 @@
       </visual>
       <collision>
+        <origin xyz="${roller_radius - roller_tangent_radius} 0 0.00925" rpy="0 0 0" />
+        <geometry>
+          <sphere radius="${roller_tangent_radius}" />
+        </geometry>
+      </collision>
+      <!-- <collision>
         <geometry>
           <mesh filename="package://armmy_omnibot/meshes/omni_wheel/Roller_Simplyfier.stl"
             scale="0.001 0.001 0.001" />
-        </geometry>
-      </collision>
-      <!-- <collision>
-        <origin xyz="0 0 0.00925" rpy="0 0 0" />
-        <geometry>
-          <cylinder radius="${roller_radius}" length="${roller_length}" />
         </geometry>
       </collision> -->

Commit message: add ground truth from gazebo for benchmark

File: armmy_omnibot/robots/newgz_omni_robot.urdf.xacro (robot description, xacro)
@@ -4,9 +4,9 @@
   <xacro:arg name="use_ros2_control" default="true" />
   <xacro:arg name="sim_mode" default="false" />
-  <xacro:include filename="$(find armmy_omnibot)/urdf/base/base.urdf.xacro"/>
-  <xacro:include filename="$(find armmy_omnibot)/urdf/omni_wheel/gz_omni_wheel.urdf.xacro"/>
-  <xacro:include filename="$(find armmy_omnibot)/urdf/lidar/lidar_gz.urdf.xacro"/>
-  <xacro:include filename="$(find armmy_omnibot)/urdf/imu/imu_gz.urdf.xacro"/>
-  <xacro:include filename="$(find armmy_omnibot)/urdf/color.xacro"/>
+  <xacro:include filename="$(find armmy_omnibot)/urdf/base/base.urdf.xacro" />
+  <xacro:include filename="$(find armmy_omnibot)/urdf/omni_wheel/gz_omni_wheel.urdf.xacro" />
+  <xacro:include filename="$(find armmy_omnibot)/urdf/lidar/lidar_gz.urdf.xacro" />
+  <xacro:include filename="$(find armmy_omnibot)/urdf/imu/imu_gz.urdf.xacro" />
+  <xacro:include filename="$(find armmy_omnibot)/urdf/color.xacro" />
   <!-- =============== Link & Joint =============== -->
   <!-- Base -->
@@ -100,4 +100,12 @@
       <parameters>$(find armmy_omnibot)/config/ros2_controller/my_controllers.yaml</parameters>
     </plugin>
+    <plugin filename="libignition-gazebo6-pose-publisher-system.so"
+      name="ignition::gazebo::systems::PosePublisher">
+      <!-- <publish_model_pose>true</publish_model_pose> -->
+      <publish_link_pose>false</publish_link_pose>
+      <publish_nested_model_pose>true</publish_nested_model_pose>
+      <!-- <static_publisher>true</static_publisher> -->
+      <static_update_frequency>10</static_update_frequency>
+   </plugin>
   </gazebo>
 </robot>

File: armmy_omnibot/urdf/roller/roller.urdf.xacro (robot description, xacro)
@@ -24,15 +24,9 @@
       </visual>
       <collision>
-        <origin xyz="${roller_radius - roller_tangent_radius} 0 0.00925" rpy="0 0 0" />
-        <geometry>
-          <sphere radius="${roller_tangent_radius}" />
-        </geometry>
-      </collision>
-      <!-- <collision>
         <geometry>
           <mesh filename="package://armmy_omnibot/meshes/omni_wheel/Roller_Simplyfier.stl"
             scale="0.001 0.001 0.001" />
         </geometry>
-      </collision> -->
+      </collision>
       <xacro:inertial_cylinder mass="${roller_mass}" length="${roller_length}"
         radius="${roller_radius}">
