Commit message: port omni robot to work with new gz

File: armmy_turtlebot3/urdf/tb3_custom_newgz/lidar.xacro (robot description, xacro)
@@ -10,5 +10,5 @@
             <origin xyz="0 0 0.0" rpy="0 0 0" />
             <geometry>
-                <mesh filename="package://turtlebot3_common/meshes/lds.dae"
+                <mesh filename="file://$(find armmy_turtlebot3)/models/turtlebot3_common/meshes/lds.dae"
                     scale="0.001 0.001 0.001" />
             </geometry>

File: armmy_turtlebot3/urdf/tb3_custom_newgz/robot_core.xacro (robot description, xacro)
@@ -58,5 +58,5 @@
             <geometry>
                 <mesh
-                    filename="package://turtlebot3_common/meshes/burger_base.dae"
+                    filename="file://$(find armmy_turtlebot3)/models/turtlebot3_common/meshes/burger_base.dae"
                     scale="0.001 0.001 0.001" />
             </geometry>
@@ -85,5 +85,5 @@
             <geometry>
                 <mesh
-                    filename="package://turtlebot3_common/meshes/tire.dae"
+                    filename="file://$(find armmy_turtlebot3)/models/turtlebot3_common/meshes/tire.dae"
                     scale="0.001 0.001 0.001" />
             </geometry>
@@ -112,5 +112,5 @@
             <geometry>
                 <mesh
-                    filename="package://turtlebot3_common/meshes/tire.dae"
+                    filename="file://$(find armmy_turtlebot3)/models/turtlebot3_common/meshes/tire.dae"
                     scale="0.001 0.001 0.001" />
             </geometry>
@@ -160,3 +160,13 @@
         <mu2 value="0.001" />
     </gazebo>
+    <gazebo>
+        <plugin
+            filename="ignition-gazebo-pose-publisher-system"
+            name="gz::sim::systems::PosePublisher">
+            <publish_link_pose>true</publish_link_pose>
+            <publish_collision_pose>false</publish_collision_pose>
+            <publish_visual_pose>false</publish_visual_pose>
+            <publish_nested_model_pose>false</publish_nested_model_pose>
+        </plugin>
+    </gazebo>
 </robot>
