Commit message: optimize mesh resulution of roller for new gazebo

File: armmy_omnibot/urdf/roller/roller.gazebo.xacro (robot description, xacro)
@@ -3,5 +3,5 @@
   <xacro:macro name="roller_gazebo_v0" params="prefix">
     <gazebo reference="${prefix}_roller_link">
-      <selfCollide>false</selfCollide>
+      <!-- <selfCollide>false</selfCollide> -->
       <mu1 value="1.2" />
       <mu2 value="1.2" />

File: armmy_omnibot/urdf/roller/roller.urdf.xacro (robot description, xacro)
@@ -24,13 +24,14 @@
       <collision>
         <geometry>
-          <mesh filename="package://armmy_omnibot/meshes/omni_wheel/roller.stl"
+          <mesh filename="package://armmy_omnibot/meshes/omni_wheel/Roller_Simplyfier.stl"
             scale="0.001 0.001 0.001" />
         </geometry>
       </collision>
-      <!-- <inertial>
-        <origin xyz="0.0 0.0 0.0" />
-        <mass value="0.02" />
-        <inertia ixx="0.000001257" ixy="0" ixz="0" iyy="0.000000342" iyz="0" izz="0.000001257" />
-      </inertial> -->
+      <!-- <collision>
+        <origin xyz="0 0 0.00925" rpy="0 0 0" />
+        <geometry>
+          <cylinder radius="${roller_radius}" length="${roller_length}" />
+        </geometry>
+      </collision> -->
       <xacro:inertial_cylinder mass="${roller_mass}" length="${roller_length}"
         radius="${roller_radius}">
@@ -49,10 +50,11 @@
           <restitution_coefficient>0.01</restitution_coefficient>
           <threshold>0</threshold>
-        </bounce>
+        </bounce> -->
         <contact>
           <ode>
             <max_vel>10</max_vel>
           </ode>
-        </contact> -->
+          <max_contacts>2</max_contacts>
+        </contact>
       </surface>
     </link>
