Commit message: finish optimised omni wheel

File: armmy_omnibot/urdf/omni_wheel/gz_omni_wheel.urdf.xacro (robot description, xacro)
@@ -22,5 +22,4 @@
                         scale="1 1 1" />
                 </geometry>
-                <!-- <material name="light_black" /> -->
             </visual>
             <xacro:inertial_cylinder mass="${wheel_mass}" length="${wheel_thickness}"
@@ -30,43 +29,35 @@
         </link>
         <xacro:roller prefix="${prefix}" num="1">
-            <!-- <origin xyz="0 0.0023125 0.0" rpy="0.0 0.0 0.0" /> -->
-            <origin xyz="0 0.004625 0.0" rpy="0.0 0.0 0.0" />
-            <!-- <origin xyz="0.015 0.1 0.0" rpy="0.0 0.0 0.0" /> -->
+            <origin xyz="0.0055 0.0046 0.0" rpy="0.0 0.0 0.0" />
             <axis xyz="0.0 0.0 1.0" />
         </xacro:roller>
-        <xacro:roller prefix="${prefix}" num="1_2">
-            <!-- <origin xyz="0 0.0023125 0.0" rpy="0.0 0.0 0.0" /> -->
-            <origin xyz="0 0.0185 0.0" rpy="0.0 0.0 0.0" />
-            <!-- <origin xyz="0.015 0.1 0.0" rpy="0.0 0.0 0.0" /> -->
-            <axis xyz="0.0 0.0 1.0" />
-        </xacro:roller>
-        <!-- <xacro:roller prefix="${prefix}" num="2">
-            <origin xyz="0.0 0.0046 0.015" rpy="-1.0 0.0 0.0" />
+        <xacro:roller prefix="${prefix}" num="2">
+            <origin xyz="0.0 0.0046 0.0055" rpy="0.0 0.0 0.0" />
             <axis xyz="-1.0 0.0 0.0" />
         </xacro:roller>
         <xacro:roller prefix="${prefix}" num="3">
-            <origin xyz="-0.015 0.0046 0.0" rpy="-0.0 0.0 -1.0" />
+            <origin xyz="-0.0055 0.0046 0.0" rpy="0.0 0.0 0.0" />
             <axis xyz="-0.0 0.0 -1.0" />
         </xacro:roller>
         <xacro:roller prefix="${prefix}" num="4">
-            <origin xyz="-0.0 0.0046 -0.015" rpy="1.0 0.0 -0.0" />
+            <origin xyz="-0.0 0.0046 -0.0055" rpy="0.0 0.0 0.0" />
             <axis xyz="1.0 0.0 -0.0" />
         </xacro:roller>
         <xacro:roller prefix="${prefix}" num="5">
-            <origin xyz="0.0106 0.0139 0.0106" rpy="-0.707107 0.0 0.707107" />
+            <origin xyz="0.0039 0.0139 0.0039" rpy="0.0 0.0 0.0" />
             <axis xyz="-0.707107 0.0 0.707107" />
         </xacro:roller>
         <xacro:roller prefix="${prefix}" num="6">
-            <origin xyz="-0.0106 0.0139 0.0106" rpy="-0.707107 0.0 -0.707107" />
+            <origin xyz="-0.0039 0.0139 0.0039" rpy="0.0 0.0 0.0" />
             <axis xyz="-0.707107 0.0 -0.707107" />
         </xacro:roller>
         <xacro:roller prefix="${prefix}" num="7">
-            <origin xyz="-0.0106 0.0139 -0.0106" rpy="0.707107 0.0 -0.707107" />
+            <origin xyz="-0.0039 0.0139 -0.0039" rpy="0.0 0.0 0.0" />
             <axis xyz="0.707107 0.0 -0.707107" />
         </xacro:roller>
         <xacro:roller prefix="${prefix}" num="8">
-            <origin xyz="0.0106 0.0139 -0.0106" rpy="0.707107 0.0 0.707107" />
+            <origin xyz="0.0039 0.0139 -0.0039" rpy="0.0 0.0 0.0" />
             <axis xyz="0.707107 0.0 0.707107" />
-        </xacro:roller> -->
+        </xacro:roller>
     </xacro:macro>
 </robot>

File: armmy_omnibot/urdf/roller/gz_roller.urdf.xacro (robot description, xacro)
@@ -2,6 +2,6 @@
 <robot xmlns:xacro="http://ros.org/wiki/xacro">
     <xacro:include filename="$(find armmy_omnibot)/urdf/inertial_macros.xacro" />
-    <xacro:property name="roller_radius" value="0.02" />
-    <xacro:property name="roller_mass" value="0.001" />
+    <xacro:property name="roller_mass" value="0.02" />
+    <xacro:property name="roller_radius" value="0.012" />
     <xacro:macro name="roller" params="prefix num *joint_origin *joint_axis">
         <link name="roller_${prefix}_${num}_link">
@@ -10,5 +10,5 @@
             </xacro:inertial_sphere>
             <collision>
-                <xacro:insert_block name="joint_origin" />
+                <origin xyz="0 0 0" rpy="0 0 0" />
                 <geometry>
                     <sphere radius="${roller_radius}" />
