Commit message: correct inertial of robot

File: armmy_omnibot/urdf/base/base.urdf.xacro (robot description, xacro)
@@ -1,49 +1,59 @@
 <?xml version="1.0"?>
 <robot xmlns:xacro="http://ros.org/wiki/xacro">
-  <xacro:include filename="$(find armmy_omnibot)/urdf/base/base.gazebo.xacro"/>
+  <xacro:include filename="$(find armmy_omnibot)/urdf/base/base.gazebo.xacro" />
+  <xacro:include filename="$(find armmy_omnibot)/urdf/inertial_macros.xacro" />
+  <xacro:property name="bass_thickness" value="0.008" />
+  <xacro:property name="base_radian" value="0.040" />
+  <xacro:property name="base_mass" value="0.05" />
   <xacro:macro name="base_v0" params="parent *joint_origin">
-	<joint name="base_link_joint" type="fixed">
-	  <xacro:insert_block name="joint_origin"/>
-	  <parent link="${parent}"/>
-	  <child link="base_link"/>
-	</joint>
-	<link name="base_link">
-	  <visual>
-		<geometry>
-		  <mesh filename="file://$(find armmy_omnibot)/meshes/base_link.stl" scale="0.001 0.001 0.001"/>
-		</geometry>
-	  </visual>
-	  <collision>
-		<geometry>
-		  <mesh filename="file://$(find armmy_omnibot)/meshes/base_link.stl" scale="0.001 0.001 0.001"/>
-		</geometry>
-	  </collision>
-	  <inertial>
+    <joint name="base_link_joint" type="fixed">
+      <xacro:insert_block name="joint_origin" />
+      <parent link="${parent}" />
+      <child link="base_link" />
+    </joint>
+    <link name="base_link">
+      <visual>
+        <geometry>
+          <mesh filename="file://$(find armmy_omnibot)/meshes/base_link.stl"
+            scale="0.001 0.001 0.001" />
+        </geometry>
+      </visual>
+      <collision>
+        <geometry>
+          <mesh filename="file://$(find armmy_omnibot)/meshes/base_link.stl"
+            scale="0.001 0.001 0.001" />
+        </geometry>
+      </collision>
+      <xacro:inertial_cylinder mass="${base_mass}" length="${bass_thickness}"
+        radius="${base_radian}">
+        <origin xyz="0 0 0" rpy="0 0 0" />
+      </xacro:inertial_cylinder>
+      <!-- <inertial>
 		<origin xyz="0 0 0"/>
 		<mass value="1.167"/>
 		<inertia ixx="0.0016" ixy="0" ixz="0" iyy="0.0016" iyz="0" izz="0.0032" />
-	  </inertial>
-          <surface>
-            <friction>
-              <ode>
-                <mu>0.8</mu>
-                <mu2>0.8</mu2>
-                <kp>1e15</kp>
-                <kd>1e13</kd>
-              </ode>
-            </friction>
-            <bounce>
-              <restitution_coefficient>0.01</restitution_coefficient>
-              <threshold>10</threshold>
-            </bounce>
-            <contact>
-              <ode>
-                <max_vel>0.01</max_vel>
-                <minDepth>0</minDepth>
-                <contact_surface_layer>0</contact_surface_layer>
-              </ode>
-            </contact>
-          </surface>
-	</link>
+	  </inertial> -->
+      <surface>
+        <friction>
+          <ode>
+            <mu>0.8</mu>
+            <mu2>0.8</mu2>
+            <kp>1e15</kp>
+            <kd>1e13</kd>
+          </ode>
+        </friction>
+        <bounce>
+          <restitution_coefficient>0.01</restitution_coefficient>
+          <threshold>10</threshold>
+        </bounce>
+        <contact>
+          <ode>
+            <max_vel>0.01</max_vel>
+            <minDepth>0</minDepth>
+            <contact_surface_layer>0</contact_surface_layer>
+          </ode>
+        </contact>
+      </surface>
+    </link>
   </xacro:macro>
 </robot>

File: armmy_omnibot/urdf/omni_wheel/omni_wheel.urdf.xacro (robot description, xacro)
@@ -3,4 +3,8 @@
   <xacro:include filename="$(find armmy_omnibot)/urdf/omni_wheel/omni_wheel.transmission.xacro"/>
   <xacro:include filename="$(find armmy_omnibot)/urdf/omni_wheel/omni_wheel.gazebo.xacro"/>
+  <xacro:include filename="$(find armmy_omnibot)/urdf/inertial_macros.xacro" />
+  <xacro:property name="wheel_thickness" value="0.0185" />
+  <xacro:property name="wheel_radian" value="0.0175" />
+  <xacro:property name="wheel_mass" value="0.05" />
   <xacro:macro name="wheel_v0" params="prefix parent *joint_origin *joint_axis">
 	<joint name="${prefix}_wheel_joint" type="continuous">
@@ -22,9 +26,13 @@
 		</geometry>
 	  </collision>
-	  <inertial>
+    <xacro:inertial_cylinder mass="${wheel_mass}" length="${wheel_thickness}"
+        radius="${wheel_radian}">
+        <origin xyz="0 ${wheel_thickness/2} 0" rpy="1.570796327 0 0" />
+      </xacro:inertial_cylinder>
+	  <!-- <inertial>
 		<origin xyz="0.0 -0.0 -0.0"/>
 		<mass value="0.25"/>
 		<inertia ixx="0.00031" ixy="0" ixz="0" iyy="0.0005" iyz="0" izz="0.00031"/>
-	  </inertial>
+	  </inertial> -->
           <surface>
             <friction>

File: armmy_omnibot/urdf/roller/roller.urdf.xacro (robot description, xacro)
@@ -1,6 +1,10 @@
 <?xml version="1.0"?>
 <robot xmlns:xacro="http://ros.org/wiki/xacro">
+  <xacro:property name="roller_length" value="0.0185" />
+  <xacro:property name="roller_radius" value="0.00475" />
+  <xacro:property name="roller_mass" value="0.005" />
   <xacro:include filename="$(find armmy_omnibot)/urdf/roller/roller.transmission.xacro" />
   <xacro:include filename="$(find armmy_omnibot)/urdf/roller/roller.gazebo.xacro" />
+  <xacro:include filename="$(find armmy_omnibot)/urdf/inertial_macros.xacro" />
   <xacro:macro name="roller_v0" params="prefix parent *joint_origin *joint_axis">
     <joint name="${prefix}_roller_joint" type="continuous">
@@ -13,27 +17,33 @@
       <visual>
         <geometry>
-          <mesh filename="package://armmy_omnibot/meshes/omni_wheel/roller.stl" scale="0.001 0.001 0.001"/>
+          <mesh filename="package://armmy_omnibot/meshes/omni_wheel/roller.stl"
+            scale="0.001 0.001 0.001" />
         </geometry>
       </visual>
       <collision>
         <geometry>
-          <mesh filename="package://armmy_omnibot/meshes/omni_wheel/roller.stl" scale="0.001 0.001 0.001" />
+          <mesh filename="package://armmy_omnibot/meshes/omni_wheel/roller.stl"
+            scale="0.001 0.001 0.001" />
         </geometry>
       </collision>
-      <inertial>
+      <!-- <inertial>
         <origin xyz="0.0 0.0 0.0" />
         <mass value="0.02" />
         <inertia ixx="0.000001257" ixy="0" ixz="0" iyy="0.000000342" iyz="0" izz="0.000001257" />
-      </inertial>
+      </inertial> -->
+      <xacro:inertial_cylinder mass="${roller_mass}" length="${roller_length}"
+        radius="${roller_radius}">
+        <origin xyz="0 0 0.00925" rpy="0 0 0" />
+      </xacro:inertial_cylinder>
       <surface>
         <friction>
           <ode>
-            <mu1>1.2</mu1>
-            <mu2>1.2</mu2>
+            <mu1>1.6</mu1>
+            <mu2>1.6</mu2>
             <kp>1e15</kp>
             <kd>1e13</kd>
           </ode>
         </friction>
-        <bounce>
+        <!-- <bounce>
           <restitution_coefficient>0.01</restitution_coefficient>
           <threshold>0</threshold>
@@ -43,5 +53,5 @@
             <max_vel>10</max_vel>
           </ode>
-        </contact>
+        </contact> -->
       </surface>
     </link>

Commit message: change baselink path

File: armmy_omnibot/urdf/base/base.urdf.xacro (robot description, xacro)
@@ -15,5 +15,5 @@
       <visual>
         <geometry>
-          <mesh filename="file://$(find armmy_omnibot)/meshes/base_link.stl"
+          <mesh filename="package://armmy_omnibot/meshes/base_link.stl"
             scale="0.001 0.001 0.001" />
         </geometry>
@@ -22,5 +22,5 @@
       <collision>
         <geometry>
-          <mesh filename="file://$(find armmy_omnibot)/meshes/base_link.stl"
+          <mesh filename="package://armmy_omnibot/meshes/base_link.stl"
             scale="0.001 0.001 0.001" />
         </geometry>

Commit message: adjust fiction of roller

File: armmy_omnibot/urdf/base/base.urdf.xacro (robot description, xacro)
@@ -5,5 +5,5 @@
   <xacro:property name="bass_thickness" value="0.008" />
   <xacro:property name="base_radian" value="0.040" />
-  <xacro:property name="base_mass" value="0.05" />
+  <xacro:property name="base_mass" value="0.2" />
   <xacro:macro name="base_v0" params="parent *joint_origin">
     <joint name="base_link_joint" type="fixed">
@@ -35,25 +35,4 @@
 		<inertia ixx="0.0016" ixy="0" ixz="0" iyy="0.0016" iyz="0" izz="0.0032" />
 	  </inertial> -->
-      <surface>
-        <friction>
-          <ode>
-            <mu>0.8</mu>
-            <mu2>0.8</mu2>
-            <kp>1e15</kp>
-            <kd>1e13</kd>
-          </ode>
-        </friction>
-        <bounce>
-          <restitution_coefficient>0.01</restitution_coefficient>
-          <threshold>10</threshold>
-        </bounce>
-        <contact>
-          <ode>
-            <max_vel>0.01</max_vel>
-            <minDepth>0</minDepth>
-            <contact_surface_layer>0</contact_surface_layer>
-          </ode>
-        </contact>
-      </surface>
     </link>
   </xacro:macro>

File: armmy_omnibot/urdf/omni_wheel/omni_wheel.urdf.xacro (robot description, xacro)
@@ -13,4 +13,5 @@
       <child link="${prefix}_wheel_link" />
       <limit effort="100" velocity="100" />
+      <dynamics damping="0.7" />
       <xacro:insert_block name="joint_axis" />
     </joint>

File: armmy_omnibot/urdf/roller/gz_roller.urdf.xacro (robot description, xacro)
@@ -15,11 +15,12 @@
                 </geometry>
             </collision>
-            <!-- <visual>
-                <xacro:insert_block name="joint_origin" />
-                <geometry>
-                    <sphere radius="${roller_radius}" />
-                </geometry>
-                <material name="Gazebo/Blue" />
-            </visual> -->
+            <surface>
+                <friction>
+                    <ode>
+                        <mu>1.0</mu>
+                        <mu2>1.0</mu2>
+                    </ode>
+                </friction>
+            </surface>
         </link>
         <joint name="roller_${prefix}_${num}_joint" type="continuous">

File: armmy_omnibot/urdf/roller/roller.gazebo.xacro (robot description, xacro)
@@ -4,5 +4,5 @@
     <gazebo reference="${prefix}_roller_link">
       <!-- <selfCollide>false</selfCollide> -->
-      <mu1 value="1.2" />
+      <mu value="8.8" />
       <mu2 value="1.2" />
     </gazebo>

File: armmy_turtlebot3/urdf/tb3_custom_newgz/ros2_control.xacro (robot description, xacro)
@@ -1,64 +1,32 @@
 <?xml version="1.0"?>
 <robot xmlns:xacro="http://www.ros.org/wiki/xacro">
-    <xacro:unless value="$(arg sim_mode)">
-        <ros2_control name="RealRobot" type="system">
-            <hardware>
-                <plugin>diffdrive_arduino/DiffDriveArduino</plugin>
-                <param name="left_wheel_name">wheel_left_joint</param>
-                <param name="right_wheel_name">wheel_right_joint</param>
-                <param name="loop_rate">30</param>
-                <param name="device">/dev/ttyUSB0</param>
-                <param name="baud_rate">57600</param>
-                <param name="timeout">1000</param>
-                <param name="enc_counts_per_rev">3436</param>
-            </hardware>
-            <joint name="wheel_left_joint">
-                <command_interface name="velocity">
-                    <param name="min">-10</param>
-                    <param name="max">10</param>
-                </command_interface>
-                <state_interface name="velocity" />
-                <state_interface name="position" />
-            </joint>
-            <joint name="wheel_right_joint">
-                <command_interface name="velocity">
-                    <param name="min">-10</param>
-                    <param name="max">10</param>
-                </command_interface>
-                <state_interface name="velocity" />
-                <state_interface name="position" />
-            </joint>
-        </ros2_control>
-    </xacro:unless>
-    <xacro:if value="$(arg sim_mode)">
-        <ros2_control name="GazeboSystem" type="system">
-            <hardware>
-                <plugin>gz_ros2_control/GazeboSimSystem</plugin>
-            </hardware>
-            <joint name="wheel_left_joint">
-                <command_interface name="velocity">
-                    <param name="min">-10</param>
-                    <param name="max">10</param>
-                </command_interface>
-                <state_interface name="velocity" />
-                <state_interface name="position" />
-            </joint>
-            <joint name="wheel_right_joint">
-                <command_interface name="velocity">
-                    <param name="min">-10</param>
-                    <param name="max">10</param>
-                </command_interface>
-                <state_interface name="velocity" />
-                <state_interface name="position" />
-            </joint>
-            <joint name="arm_joint">
-                <command_interface name="position" />
-                <state_interface name="position">
-                    <param name="initial_value">0.0</param>
-                </state_interface>
-                <state_interface name="velocity" />
-            </joint>
-        </ros2_control>
-    </xacro:if>
+    <ros2_control name="GazeboSystem" type="system">
+        <hardware>
+            <plugin>gz_ros2_control/GazeboSimSystem</plugin>
+        </hardware>
+        <joint name="wheel_left_joint">
+            <command_interface name="velocity">
+                <param name="min">-10</param>
+                <param name="max">10</param>
+            </command_interface>
+            <state_interface name="velocity" />
+            <state_interface name="position" />
+        </joint>
+        <joint name="wheel_right_joint">
+            <command_interface name="velocity">
+                <param name="min">-10</param>
+                <param name="max">10</param>
+            </command_interface>
+            <state_interface name="velocity" />
+            <state_interface name="position" />
+        </joint>
+        <joint name="arm_joint">
+            <command_interface name="position" />
+            <state_interface name="position">
+                <param name="initial_value">0.0</param>
+            </state_interface>
+            <state_interface name="velocity" />
+        </joint>
+    </ros2_control>
     <gazebo>
         <plugin name="gz_ros2_control::GazeboSimROS2ControlPlugin"
